File: IIITDuino_hemanth/IIITDuino Ver0.5.brd (EAGLE design)
At the start: 100 x 81.7 mm, 86 parts, among them IC3 LM1117, J2 DCJ0202, M1 ELECTRET_MICROPHON-TOM-1545P-R, Q1 ZXMP6A13FTA, Q2 2N7002PW, T1 BC547, U1 FT231XS, U2 MIC5205, U4 ATMEGA328P_PDIP, Y1 16MHz

Commit message: Seggregated the boards
Parts:
- removed FRAME2: FRAME-LETTER, SparkFun-Aesthetics:CREATIVE_COMMONS
